File: Versions/LED-CLOCK 1.0/Projeto_Relogio_LED.sch (EAGLE design)
At the start: 68 parts, among them IC1 NE555, IC10 74HC393D, IC11 4081D, IC2 4056N, IC3 4056N, IC4 4056N, IC5 4056N, IC6 4056N, IC7 4056N, IC8 74HC393D, IC9 74HC393D, T1 BD239, X1 4AND, X10 INVERTER, X11 DFF, X12 DFF, X13 DFF, X14 DFF, X15 DFF, X16 DFF, X17 DFF, X18 DFF, X19 DFF, X2 4AND, X20 DFF, X21 DFF, X22 DFF, X23 INVERTER, X24 INVERTER, X25 INVERTER, X26 INVERTER, X27 INVERTER, X28 INVERTER, X29 INVERTER, X3 4AND, X30 INVERTER, X31 4AND, X32 4AND, X33 4AND, X34 3AND, X35 AND, X4 4AND, X5 INVERTER, X6 INVERTER, X7 4AND, X9 INVERTER

Commit message: docs
Parts:
- removed TOMADA_127V: (no value), con-ptr500:AK500/2-H
- added FONTE_AC: 350428-1, con-amp:350428-1
Connections:
- net GND: now also FONTE_AC.1; no longer TOMADA_127V-2.KL
- net VCC: now also FONTE_AC.2; no longer TOMADA_127V-1.KL
Changed lines of the file:
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@@
 <part name="X28" library="ngspice-digital" library_urn="urn:adsk.eagle:library:5610454" deviceset="INVERTER" device=""/>
 <part name="X29" library="ngspice-digital" library_urn="urn:adsk.eagle:library:5610454" deviceset="INVERTER" device=""/>
-<part name="TOMADA_127V" library="con-ptr500" library_urn="urn:adsk.eagle:library:181" deviceset="AK500/2-H" device="" package3d_urn="urn:adsk.eagle:package:9901/1"/>
 <part name="GND1" library="audio amplifier example" library_urn="urn:adsk.eagle:library:970892" deviceset="GND" device="" value="SUP"/>
 <part name="GND2" library="audio amplifier example" library_urn="urn:adsk.eagle:library:970892" deviceset="GND" device="" value="SUP"/>
@@
 <part name="X34" library="ngspice-digital" library_urn="urn:adsk.eagle:library:5610454" deviceset="3AND" device=""/>
 <part name="X35" library="ngspice-digital" library_urn="urn:adsk.eagle:library:5610454" deviceset="AND" device=""/>
+<part name="FONTE_AC" library="con-amp" library_urn="urn:adsk.eagle:library:127" deviceset="350428-1" device="" package3d_urn="urn:adsk.eagle:package:8081751/1"/>
 </parts>
 <sheets>
@@
 <attribute name="VALUE" x="210.82" y="124.46" size="1.778" layer="96" rot="MR270"/>
 </instance>
-<instance part="TOMADA_127V" gate="-1" x="10.16" y="63.5" smashed="yes">
-<attribute name="NAME" x="8.89" y="64.389" size="1.778" layer="95" rot="R180"/>
-</instance>
-<instance part="TOMADA_127V" gate="-2" x="10.16" y="50.8" smashed="yes">
-<attribute name="NAME" x="8.89" y="51.689" size="1.778" layer="95" rot="R180"/>
-<attribute name="VALUE" x="6.35" y="47.117" size="1.778" layer="96"/>
-</instance>
 <instance part="GND1" gate="G$1" x="15.24" y="50.8" smashed="yes"/>
 <instance part="GND2" gate="G$1" x="20.32" y="50.8" smashed="yes"/>
@@
 <attribute name="NAME" x="406.4" y="80.01" size="1.778" layer="95"/>
 <attribute name="VALUE" x="406.4" y="66.04" size="1.778" layer="96"/>
+</instance>
+<instance part="FONTE_AC" gate="G$1" x="2.54" y="55.88" smashed="yes" rot="R90">
+<attribute name="NAME" x="2.54" y="60.96" size="1.778" layer="95" rot="R90"/>
+<attribute name="VALUE" x="6.35" y="60.96" size="1.778" layer="96" rot="R90"/>
 </instance>
 </instances>
@@
 <segment>
 <pinref part="TR1" gate="G$1" pin="1"/>
-<pinref part="TOMADA_127V" gate="-2" pin="KL"/>
 <pinref part="GND1" gate="G$1" pin="GND"/>
+<pinref part="FONTE_AC" gate="G$1" pin="1"/>
+<wire x1="5.08" y1="55.88" x2="5.08" y2="50.8" width="0.1524" layer="91"/>
+<wire x1="5.08" y1="50.8" x2="15.24" y2="50.8" width="0.1524" layer="91"/>
 <junction x="15.24" y="50.8"/>
 </segment>
@@
 <segment>
 <pinref part="TR1" gate="G$1" pin="2"/>
-<pinref part="TOMADA_127V" gate="-1" pin="KL"/>
 <pinref part="P+1" gate="VCC" pin="VCC"/>
+<pinref part="FONTE_AC" gate="G$1" pin="2"/>
+<wire x1="5.08" y1="58.42" x2="5.08" y2="63.5" width="0.1524" layer="91"/>
+<wire x1="5.08" y1="63.5" x2="15.24" y2="63.5" width="0.1524" layer="91"/>
 <junction x="15.24" y="63.5"/>
 </segment>

Commit message: docs
Parts:
- removed X1, X2, X3, X4, X7: 4AND, ngspice-digital:4AND
- removed X10, X24, X25, X26, X27, X28, X29, X30, X5, X6, X9: INVERTER, ngspice-digital:INVERTER
- added IC12, IC13, IC14, IC15, IC16: 74AHC1G08DCK, 74xx-little-us:74AHC1G08DCK
Connections:
- removed net N$112: X2.B, X24.O
- removed net N$113: X2.A, X25.O
- removed net N$115: X26.O, X4.B
- removed net N$116: X27.O, X4.A
- removed net N$118: X28.O, X3.C
- removed net N$119: X29.O, X3.B
- removed net N$120: IC11A.I0, X30.O
- removed net N$121: X10.O, X7.C
- removed net N$122: IC10B.A, X7.Y
- removed net N$67: IC5A.I3, IC8B.QD, X2.C
- removed net N$91: X1.C, X6.O
- net N$1: now also IC13A.O; no longer X1.Y
- net N$107: now also IC11A.I0
- net N$114: now also IC16A.O; no longer X4.Y
- net N$117: now also IC14A.O; no longer X3.Y
- net N$2: now also IC15A.I1, IC5A.I3, IC8B.QD; no longer X1.A, X5.O
- net N$3: now also IC15A.O; no longer X2.Y
- net N$63: no longer X27.I
- net N$64: no longer X26.I
- net N$65: now also IC16A.I1; no longer X4.C
- net N$66: now also IC16A.I0; no longer X4.D
- net N$68: no longer X25.I
- net N$69: no longer X24.I
- net N$70: now also IC15A.I0; no longer X2.D
- net N$71: now also IC14A.I1; no longer X3.A
- net N$72: no longer X29.I
- net N$73: no longer X28.I
- net N$74: now also IC14A.I0; no longer X3.D
- net N$75: now also IC13A.I1; no longer X1.D
- net N$76: no longer X6.I
- net N$77: now also IC13A.I0; no longer X1.B
- net N$78: no longer X5.I
- net N$79: now also IC12A.I1; no longer X7.D
- net N$80: no longer X10.I
- net N$81: now also IC12A.I0; no longer IC11A.I1, X7.B
- net N$82: now also IC11A.I1; no longer X30.I, X9.I
- net N$92: now also IC10B.A, IC12A.O; no longer X7.A, X9.O
Other:
- moved on the sheet: D5, D7, D8, D9, DS1, DS2, DS3, DS4, DS5, DS6, IC2, IC3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

Commit message: docs
Parts:
- IC11: value 4081D -> 74AHC1G08DCK; device 40xx:4081D -> 74xx-little-us:74AHC1G08DCK
Connections:
- removed net N$123: IC11A.O, IC11B.I0
- removed net N$125: X18.Q, X33.D
- new net N$67: X18.Q, X33.A
- net N$10: no longer X31.A
- net N$102: now also X33.D; no longer X33.A
- net N$103: now also X32.B
- net N$104: now also X32.A
- net N$107: no longer IC11A.I0, S1.P
- net N$11: no longer X31.B
- net N$111: now also IC11A.O; no longer IC11B.O
- net N$12: no longer X31.C
- net N$13: no longer X31.D
- net N$14: now also X32.D; no longer X32.A
- net N$15: now also S1.P; no longer X32.B
- net N$16: no longer X32.C
- net N$17: no longer X32.D
- net N$19: now also X33.C; no longer X33.B
- net N$20: now also X33.B; no longer X33.C
- net N$81: now also IC11A.I0
- net N$82: no longer IC11A.I1
- net N$86: now also IC11A.I1; no longer IC11B.I1
- net N$93: now also X31.D
- net N$94: now also X31.C
- net N$95: now also X31.B
- net N$96: now also X31.A
- net N$98: now also X32.C
