File: Versions/LED-CLOCK 1.0/Modulo 1/Projeto_Relogio_LED.brd (EAGLE design)
At the start: 160 x 100 mm, 15 parts, among them IC1 NE555, T1 BD239

Commit message: update
Ultima versão para impressão na placa
Parts:
- removed C2: 200uF, rcl:C025-024X044
- removed C4: 250mF, rcl:C025-024X044
- removed C5: 10nF, rcl:C025-024X044
- removed D1, D2, D3, D4: 1N4004, diode:DO41-10
- removed D6: 1N4728, diode:DO41Z10
- removed FONTE_AC: 350428-1, con-amp:350428-1
- removed R3: 10K, Tinkercad:RESAD1016W63L850D250B
- removed R4: 100K, Tinkercad:RESAD1016W63L850D250B
- removed T1: BD239, transistor:TO220
- removed TR1: 10W, inductor-neosid:U15
- added CLOCLK_3600HZ: 350428-1, con-amp:350428-1
- added D12, D13, D14: 1N4004, diode:DO41-10
- added D5, D7, D8, D9: HLMP6, display-hp:HLMP6
- added DS1, DS2, DS3, DS4, DS5, DS6: ACSA56-51SUR, Display_LED:ACSA56-51SURKWA
- added IC10, IC8, IC9: 74HC393D, 74xx-eu:SO14
- added IC11, IC12, IC13, IC14, IC15, IC16: 74AHC1G08DCK, 74xx-little-us:SC70-5
- added IC17, IC18: 74AC21D, 74xx-eu:SO14
- added IC19: 74HC11N, 74xx-eu:DIL14
- added IC2, IC3, IC4, IC5, IC6, IC7: 4056N, 40xx:DIL16
- added IC20: 4069D, 40xx:SO14
- added IC21, IC22, IC23, IC24, IC25, IC26: 4013D, 40xx:SO14
- added R2: 100, Tinkercad:RESAD1016W63L850D250B
- added S1, S3: (no value), switch-omron:B3F-10XX
- IC1: value NE555 -> 74AHC1G08DCK; device st-microelectronics:DIL-08 -> 74xx-little-us:SC70-5
- R1: value 1K -> 100
- moved IC1 88.8 mm to (7.62, 33.0)
- moved R1 37.7 mm to (52.1, 74.9), turned to 90 degrees
Connections:
- new net N$100: IC17.9, IC21.2, IC21.5
- new net N$105: D12.C, D13.C, D14.C, IC1.1, IC1.2, IC8.13
- new net N$106: IC17.8, IC19.1
- new net N$107: R1.2, R2.2
- new net N$108: D13.A, S1.1
- new net N$109: D14.A, S3.1
- new net N$110: IC18.6, IC19.2
- new net N$111: IC1.4, IC10.12, IC10.2, IC11.4, IC8.12, IC8.2, IC9.12, IC9.2
- new net N$112: IC17.1, IC26.13
- new net N$113: CLOCLK_3600HZ.1, D7.K, D9.K, DS1.3, DS1.8, DS2.3, DS2.8, DS3.3, DS3.8, DS4.3, DS4.8, DS5.3, DS5.8, DS6.3, DS6.8
- new net N$114: IC16.4, IC9.1
- new net N$115: IC17.2, IC26.2, IC26.5
- new net N$117: IC14.4, IC9.13
- new net N$12: IC22.13, IC23.3
- new net N$124: IC17.6, IC19.13
- new net N$13: IC23.1, IC23.11
- new net N$14: IC24.1, IC24.11
- new net N$15: IC18.4, IC24.2, IC24.5
- new net N$16: IC24.13, IC25.3
- new net N$17: IC25.1, IC25.11
- new net N$18: IC17.4, IC25.13, IC26.3
- new net N$19: IC26.1, IC26.11
- new net N$20: IC23.13, IC24.3
- new net N$21: DS5.7, IC7.9
- new net N$22: DS5.6, IC7.10
- new net N$23: DS5.4, IC7.11
- new net N$24: DS5.2, IC7.12
- new net N$25: DS5.1, IC7.13
- new net N$26: DS5.10, DS5.5, IC7.14
- new net N$27: DS5.9, IC7.15
- new net N$28: DS6.7, IC6.9
- new net N$29: DS6.6, IC6.10
- new net N$30: DS6.4, IC6.11
- new net N$31: DS6.2, IC6.12
- new net N$32: DS6.1, IC6.13
- new net N$33: DS6.10, DS6.5, IC6.14
- new net N$34: DS6.9, IC6.15
- new net N$35: DS3.7, IC5.9
- new net N$36: DS3.6, IC5.10
- new net N$37: DS3.4, IC5.11
- new net N$38: DS3.2, IC5.12
- new net N$39: DS3.1, IC5.13
- new net N$40: DS3.10, DS3.5, IC5.14
- new net N$41: DS3.9, IC5.15
- new net N$42: DS4.7, IC4.9
- new net N$43: DS4.6, IC4.10
- new net N$44: DS4.4, IC4.11
- new net N$45: DS4.2, IC4.12
- new net N$46: DS4.1, IC4.13
- new net N$47: DS4.10, DS4.5, IC4.14
- new net N$48: DS4.9, IC4.15
- new net N$49: DS1.7, IC3.9
- new net N$50: DS1.6, IC3.10
- new net N$51: DS1.4, IC3.11
- new net N$52: DS1.2, IC3.12
- new net N$53: DS1.1, IC3.13
- new net N$54: DS1.10, DS1.5, IC3.14
- new net N$55: DS1.9, IC3.15
- new net N$56: DS2.7, IC2.9
- new net N$57: DS2.6, IC2.10
- new net N$58: DS2.4, IC2.11
- new net N$59: DS2.2, IC2.12
- new net N$60: DS2.1, IC2.13
- new net N$61: DS2.10, DS2.5, IC2.14
- new net N$62: DS2.9, IC2.15
- new net N$63: IC4.4, IC8.6
- new net N$64: IC4.2, IC8.5
- new net N$65: IC16.2, IC4.3, IC8.4
- new net N$66: IC16.1, IC4.5, IC8.3
- new net N$68: IC5.2, IC8.9
- new net N$69: IC5.3, IC8.10
- new net N$70: IC15.1, IC5.5, IC8.11
- new net N$71: IC14.2, IC3.4, IC9.6
- new net N$72: IC3.2, IC9.5
- new net N$73: IC3.3, IC9.4
- new net N$74: IC14.1, IC3.5, IC9.3
- new net N$75: IC13.2, IC2.4, IC9.8
- new net N$76: IC2.2, IC9.9
- new net N$77: IC13.1, IC2.3, IC9.10
- new net N$78: IC2.5, IC9.11
- new net N$79: IC10.6, IC12.2, IC7.4
- new net N$8: IC21.1, IC21.11
- new net N$80: IC10.5, IC7.2
- new net N$81: IC10.4, IC11.1, IC12.1, IC7.3
- new net N$82: IC10.3, IC7.5
- new net N$83: IC10.8, IC6.4
- new net N$84: IC10.9, IC6.2
- new net N$85: IC10.10, IC6.3
- new net N$86: IC10.11, IC11.2, IC6.5
- new net N$87: D5.K, D7.A
- new net N$88: D8.K, D9.A
- new net N$89: IC17.10, IC21.12, IC21.9
- new net N$90: IC22.2, IC22.5
- new net N$91: IC17.13, IC22.12, IC22.9
- new net N$92: IC10.13, IC12.4
- new net N$93: IC18.1, IC23.2, IC23.5
- new net N$94: IC18.2, IC23.12, IC23.9
- new net N$95: IC18.5, IC24.12, IC24.9
- new net N$96: IC17.5, IC25.2, IC25.5
- new net N$97: IC25.12, IC25.9
- new net N$99: IC26.12, IC26.9
- new net VCC: IC1.5, IC10.14, IC11.5, IC12.5, IC13.5, IC14.5, IC15.5, IC16.5, IC17.14, IC18.14, IC19.14, IC2.16, IC3.16, IC4.16, IC5.16, IC6.16, IC7.16, IC8.14, IC9.14
- new net VDD: IC20.14, IC21.14, IC22.14, IC23.14, IC24.14, IC25.14, IC26.14
- new net VEE: IC2.7, IC3.7, IC4.7, IC5.7, IC6.7, IC7.7
- new net VSS: IC20.7, IC21.7, IC22.7, IC23.7, IC24.7, IC25.7, IC26.7
- net GND: now also IC1.3, IC10.7, IC11.3, IC12.3, IC13.3, IC14.3, IC15.3, IC16.3, IC17.7, IC18.7, IC19.7, IC2.8, IC3.8, IC4.8, IC5.8, IC6.8, IC7.8, IC8.7, IC9.7; no longer C2.1, C4.2, C5.2, D3.A, D4.A, D6.A, IC1.1
- net N$1: now also IC10.1, IC13.4; no longer C5.1, IC1.5
- net N$10: now also IC21.13, IC22.3; no longer C4.1, IC1.2, IC1.6, R4.2
- net N$11: now also IC17.12, IC22.1, IC22.11; no longer D6.C, R1.2, T1.1
- net N$2: now also IC15.2, IC5.4, IC8.8; no longer FONTE_AC.2, TR1.2
- net N$3: now also IC15.4, IC8.1; no longer FONTE_AC.1, TR1.1
- net N$4: now also D5.A, R2.1; no longer D1.A, D3.C, TR1.4
- net N$5: now also D8.A, R1.1; no longer IC1.4, IC1.8, R3.2, T1.3
- net N$6: now also D12.A, IC19.12; no longer IC1.7, R3.1, R4.1
- net N$7: now also IC20.2, IC21.3, S1.3; no longer D2.A, D4.C, TR1.3
- net N$9: now also CLOCLK_3600HZ.2, IC20.1, S3.3; no longer C2.2, D1.C, D2.C, R1.1, T1.2
Other:
- board size 160 x 100 mm -> 251.4 x 78.4 mm

Commit message: chore
Parts:
- removed IC12, IC13, IC14, IC15, IC16: 74AHC1G08DCK, 74xx-little-us:SC70-5
- IC1, IC11: value 74AHC1G08DCK -> 74AC08N; device 74xx-little-us:SC70-5 -> 74xx-eu:DIL14
- IC10, IC8, IC9: value 74HC393D -> 74AC393N; device 74xx-eu:SO14 -> 74xx-eu:DIL14
- IC17, IC18: value 74AC21D -> 74AC21N; device 74xx-eu:SO14 -> 74xx-eu:DIL14
- IC20: value 4069D -> 4069N; device 40xx:SO14 -> 40xx:DIL14
- IC21, IC22, IC23, IC24, IC25, IC26: value 4013D -> 4013N; device 40xx:SO14 -> 40xx:DIL14
- moved IC18 139.3 mm to (161.3, 49.5)
- moved IC11 121.8 mm to (47.0, 54.6)
- moved D12 83.6 mm to (154.9, 10.2)
- moved D13 83.6 mm to (161.3, 10.2)
- moved S1 83.6 mm to (154.9, -8.89)
- moved S3 83.6 mm to (165.1, -8.89)
- moved D14 83.6 mm to (167.6, 10.2)
- moved IC19 72.5 mm to (132.1, 10.2)
- moved IC21 71.2 mm to (68.6, 11.4)
- moved IC17 69.0 mm to (105.4, 10.2)
- moved IC1 64.7 mm to (-53.3, 54.6), turned to 0 degrees
- moved IC26 57.6 mm to (-108.0, 11.4)
- moved CLOCLK_3600HZ 52.2 mm to (-148.6, -10.2)
- moved DS3 51.8 mm to (160.0, 86.4)
- moved IC20 47.6 mm to (-127.0, -6.35)
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Connections:
- removed net N$107: R1.2, R2.2
- net GND: now also IC1.7, IC11.7; no longer IC1.3, IC11.3, IC12.3, IC13.3, IC14.3, IC15.3, IC16.3
- net N$1: now also IC1.8; no longer IC13.4
- net N$105: now also IC11.4, IC11.5; no longer IC1.1, IC1.2
- net N$111: now also IC1.3, IC11.6; no longer IC1.4, IC11.4
- net N$114: now also IC11.3; no longer IC16.4
- net N$117: now also IC1.11; no longer IC14.4
- net N$2: now also IC11.10; no longer IC15.2
- net N$3: now also IC11.8; no longer IC15.4
- net N$65: now also IC11.2; no longer IC16.2
- net N$66: now also IC11.1; no longer IC16.1
- net N$70: now also IC11.9; no longer IC15.1
- net N$71: now also IC1.13; no longer IC14.2
- net N$74: now also IC1.12; no longer IC14.1
- net N$75: now also IC1.10; no longer IC13.2
- net N$77: now also IC1.9; no longer IC13.1
- net N$79: now also IC1.5; no longer IC12.2
- net N$81: now also IC1.1, IC1.4; no longer IC11.1, IC12.1
- net N$86: now also IC1.2; no longer IC11.2
- net N$9: now also R1.2, R2.2
- net N$92: now also IC1.6; no longer IC12.4
- net VCC: now also IC1.14, IC11.14; no longer IC1.5, IC11.5, IC12.5, IC13.5, IC14.5, IC15.5, IC16.5
Routing:
- net GND: track 0.00 -> 916.8 mm
- net VCC: track 0.00 -> 901.8 mm
- net N$9: track 0.00 -> 687.6 mm
- net N$18: track 0.00 -> 606.0 mm
- net N$7: track 0.00 -> 544.8 mm
- net N$94: track 0.00 -> 333.4 mm
- net VDD: track 0.00 -> 258.7 mm
- net N$111: track 0.00 -> 247.4 mm
- net N$89: track 0.00 -> 238.0 mm
- net N$105: track 0.00 -> 237.1 mm
- net VSS: track 0.00 -> 208.9 mm
- net N$71: track 0.00 -> 166.7 mm
- net N$74: track 0.00 -> 162.9 mm
- net N$78: track 0.00 -> 161.5 mm
- net N$66: track 0.00 -> 128.5 mm
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Other:
- board size 251.4 x 78.4 mm -> 328.9 x 131.8 mm

Commit message: docs
Parts:
- removed DS1, DS2, DS3, DS4, DS5, DS6: ACSA56-51SUR, Display_LED:ACSA56-51SURKWA
- added LED1, LED2, LED3, LED4, LED5, LED6: S4301B, led-7-segment:S4301B
Connections:
- net N$113: now also LED1.3, LED1.8, LED2.3, LED2.8, LED3.3, LED3.8, LED4.3, LED4.8, LED5.3, LED5.8, LED6.3, LED6.8; no longer DS1.3, DS1.8, DS2.3, DS2.8, DS3.3, DS3.8, DS4.3, DS4.8, DS5.3, DS5.8, DS6.3, DS6.8
- net N$21: now also IC7.14, LED6.1; no longer DS5.7, IC7.9
- net N$22: now also IC7.15, LED6.2; no longer DS5.6, IC7.10
- net N$23: now also IC7.13, LED6.4; no longer DS5.4, IC7.11
- net N$24: now also LED6.5; no longer DS5.2
- net N$25: now also IC7.11, LED6.7; no longer DS5.1, IC7.13
- net N$26: now also IC7.10, LED6.9; no longer DS5.10, DS5.5, IC7.14
- net N$27: now also IC7.9, LED6.10; no longer DS5.9, IC7.15
- net N$28: now also LED1.10; no longer DS6.7
- net N$29: now also LED1.9; no longer DS6.6
- net N$30: now also LED1.7; no longer DS6.4
- net N$31: now also LED1.5; no longer DS6.2
- net N$32: now also LED1.4; no longer DS6.1
- net N$33: now also IC6.15, LED1.2; no longer DS6.10, DS6.5, IC6.14
- net N$34: now also IC6.14, LED1.1; no longer DS6.9, IC6.15
- net N$35: now also IC2.14, LED5.1; no longer DS3.7, IC5.9
- net N$36: now also IC2.15, LED5.2; no longer DS3.6, IC5.10
- net N$37: now also IC2.13, LED5.4; no longer DS3.4, IC5.11
- net N$38: now also IC2.12, LED5.5; no longer DS3.2, IC5.12
- net N$39: now also IC2.11, LED5.7; no longer DS3.1, IC5.13
- net N$40: now also IC2.10, LED5.9; no longer DS3.10, DS3.5, IC5.14
- net N$41: now also IC2.9, LED5.10; no longer DS3.9, IC5.15
- net N$42: now also IC3.9, LED4.10; no longer DS4.7, IC4.9
- net N$43: now also IC3.10, LED4.9; no longer DS4.6, IC4.10
- net N$44: now also IC3.11, LED4.7; no longer DS4.4, IC4.11
- net N$45: now also IC3.12, LED4.5; no longer DS4.2, IC4.12
- net N$46: now also IC3.13, LED4.4; no longer DS4.1, IC4.13
- net N$47: now also IC3.15, LED4.2; no longer DS4.10, DS4.5, IC4.14
- net N$48: now also IC3.14, LED4.1; no longer DS4.9, IC4.15
- net N$49: now also IC4.14, LED3.1; no longer DS1.7, IC3.9
- net N$50: now also IC4.15, LED3.2; no longer DS1.6, IC3.10
- net N$51: now also IC4.13, LED3.4; no longer DS1.4, IC3.11
- net N$52: now also IC4.12, LED3.5; no longer DS1.2, IC3.12
- net N$53: now also IC4.11, LED3.7; no longer DS1.1, IC3.13
- net N$54: now also IC4.10, LED3.9; no longer DS1.10, DS1.5, IC3.14
- net N$55: now also IC4.9, LED3.10; no longer DS1.9, IC3.15
- net N$56: now also IC5.14, LED2.1; no longer DS2.7, IC2.9
- net N$57: now also IC5.15, LED2.2; no longer DS2.6, IC2.10
- net N$58: now also IC5.13, LED2.4; no longer DS2.4, IC2.11
- net N$59: now also IC5.12, LED2.5; no longer DS2.2, IC2.12
- net N$60: now also IC5.11, LED2.7; no longer DS2.1, IC2.13
- net N$61: now also IC5.10, LED2.9; no longer DS2.10, DS2.5, IC2.14
- net N$62: now also IC5.9, LED2.10; no longer DS2.9, IC2.15
Routing:
- net N$113: track 0.00 -> 683.8 mm, vias 0 -> 2
- net N$18: track 606.0 -> 93.9 mm, vias 0 -> 2
- net VCC: track 901.8 -> 1176.1 mm
- net N$7: track 544.8 -> 298.1 mm, vias 0 -> 2
- net N$94: track 333.4 -> 92.5 mm, vias 0 -> 2
- net N$89: track 238.0 -> 60.0 mm
- net N$71: track 166.7 -> 18.7 mm, vias 0 -> 3
- net N$74: track 162.9 -> 17.7 mm, vias 0 -> 3
- net N$78: track 161.5 -> 44.0 mm
- net N$91: track 9.20 -> 103.5 mm, vias 0 -> 2
- net N$2: track 113.2 -> 26.5 mm, vias 0 -> 3
- net GND: track 916.8 -> 839.4 mm
- net N$95: track 9.20 -> 86.5 mm, vias 0 -> 2
- net N$75: track 104.0 -> 30.8 mm, vias 0 -> 3
- net N$70: track 128.3 -> 56.8 mm, vias 0 -> 4
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- added copper zone on layer 16, net GND
Other:
- board size 328.9 x 131.8 mm -> 330.2 x 131.8 mm
