File: Versions/LED-CLOCK 1.0/Modulo 1/Projeto_Relogio_LED.sch (EAGLE design)
At the start: 15 parts, among them IC1 NE555, T1 BD239

Commit message: update docs
Parts:
- TR1: value (none) -> 10W
Connections:
- removed net N$10 (its old number): IC1.OUT

Commit message: update
Ultima versão para impressão na placa
Parts:
- removed C2: 200uF, rcl:C-EU025-024X044
- removed C4: 250mF, rcl:C-EU025-024X044
- removed C5: 10nF, rcl:C-EU025-024X044
- removed D1, D2, D3, D4: 1N4004, diode:1N4004
- removed D6: 1N4728, diode:1N4728
- removed FONTE_AC: 350428-1, con-amp:350428-1
- removed R3: 10K, Tinkercad:RESISTOR_AXIAL-10.16MM-PITCH
- removed R4: 100K, Tinkercad:RESISTOR_AXIAL-10.16MM-PITCH
- removed T1: BD239, transistor:BD239
- removed TR1: 10W, inductor-neosid:U15-TRANSFORMER
- added CLOCLK_3600HZ: 350428-1, con-amp:350428-1
- added D12, D13, D14: 1N4004, diode:1N4004
- added D5, D7, D8, D9: HLMP6, display-hp:HLMP6
- added DS1, DS2, DS3, DS4, DS5, DS6: ACSA56-51SUR, Display_LED:ACSA56-51SUR
- added IC10, IC8, IC9: 74HC393D, 74xx-eu:74HC393D
- added IC11, IC12, IC13, IC14, IC15, IC16: 74AHC1G08DCK, 74xx-little-us:74AHC1G08DCK
- added IC17, IC18: 74AC21D, 74xx-eu:74AC21D
- added IC19: 74HC11N, 74xx-eu:74HC11N
- added IC2, IC3, IC4, IC5, IC6, IC7: 4056N, 40xx:4056N
- added IC20: 4069D, 40xx:4069D
- added IC21, IC22, IC23, IC24, IC25, IC26: 4013D, 40xx:4013D
- added R2: 100, Tinkercad:RESISTOR_AXIAL-10.16MM-PITCH
- added S1, S3: (no value), switch-omron:10-XX
- IC1: value NE555 -> 74AHC1G08DCK; device st-microelectronics:NE555 -> 74xx-little-us:74AHC1G08DCK
- R1: value 1K -> 100
Connections:
- removed net GND: C2.1, C4.2, C5.2, D3.A, D4.A, D6.A, IC1.GND
- new net N$100: IC17B.I0, IC21A.!Q, IC21A.D
- new net N$105: D12.C, D13.C, D14.C, IC1A.I0, IC1A.I1, IC8B.A
- new net N$106: IC17B.O, IC19A.I0
- new net N$107: R1.2, R2.2
- new net N$108: D13.A, S1.S
- new net N$109: D14.A, S3.S
- new net N$110: IC18A.O, IC19A.I1
- new net N$111: IC10A.CLR, IC10B.CLR, IC11A.O, IC1A.O, IC8A.CLR, IC8B.CLR, IC9A.CLR, IC9B.CLR
- new net N$112: IC17A.I0, IC26B.Q
- new net N$113: CLOCLK_3600HZ.1, D7.K, D9.K, DS1.COM1, DS2.COM1, DS3.COM1, DS4.COM1, DS5.COM1, DS6.COM1
- new net N$114: IC16A.O, IC9A.A
- new net N$115: IC17A.I1, IC26A.!Q, IC26A.D
- new net N$117: IC14A.O, IC9B.A
- new net N$12: IC22B.Q, IC23A.CLK
- new net N$124: IC17A.O, IC19A.I2
- new net N$13: IC23A.Q, IC23B.CLK
- new net N$14: IC24A.Q, IC24B.CLK
- new net N$15: IC18A.I2, IC24A.!Q, IC24A.D
- new net N$16: IC24B.Q, IC25A.CLK
- new net N$17: IC25A.Q, IC25B.CLK
- new net N$18: IC17A.I2, IC25B.Q, IC26A.CLK
- new net N$19: IC26A.Q, IC26B.CLK
- new net N$20: IC23B.Q, IC24A.CLK
- new net N$21: DS5.A, IC7A.A
- new net N$22: DS5.B, IC7A.B
- new net N$23: DS5.C, IC7A.C
- new net N$24: DS5.D, IC7A.D
- new net N$25: DS5.E, IC7A.E
- new net N$26: DS5.G, IC7A.G
- new net N$27: DS5.F, IC7A.F
- new net N$28: DS6.A, IC6A.A
- new net N$29: DS6.B, IC6A.B
- new net N$30: DS6.C, IC6A.C
- new net N$31: DS6.D, IC6A.D
- new net N$32: DS6.E, IC6A.E
- new net N$33: DS6.G, IC6A.G
- new net N$34: DS6.F, IC6A.F
- new net N$35: DS3.A, IC5A.A
- new net N$36: DS3.B, IC5A.B
- new net N$37: DS3.C, IC5A.C
- new net N$38: DS3.D, IC5A.D
- new net N$39: DS3.E, IC5A.E
- new net N$40: DS3.G, IC5A.G
- new net N$41: DS3.F, IC5A.F
- new net N$42: DS4.A, IC4A.A
- new net N$43: DS4.B, IC4A.B
- new net N$44: DS4.C, IC4A.C
- new net N$45: DS4.D, IC4A.D
- new net N$46: DS4.E, IC4A.E
- new net N$47: DS4.G, IC4A.G
- new net N$48: DS4.F, IC4A.F
- new net N$49: DS1.A, IC3A.A
- new net N$50: DS1.B, IC3A.B
- new net N$51: DS1.C, IC3A.C
- new net N$52: DS1.D, IC3A.D
- new net N$53: DS1.E, IC3A.E
- new net N$54: DS1.G, IC3A.G
- new net N$55: DS1.F, IC3A.F
- new net N$56: DS2.A, IC2A.A
- new net N$57: DS2.B, IC2A.B
- new net N$58: DS2.C, IC2A.C
- new net N$59: DS2.D, IC2A.D
- new net N$60: DS2.E, IC2A.E
- new net N$61: DS2.G, IC2A.G
- new net N$62: DS2.F, IC2A.F
- new net N$63: IC4A.I3, IC8A.QD
- new net N$64: IC4A.I2, IC8A.QC
- new net N$65: IC16A.I1, IC4A.I1, IC8A.QB
- new net N$66: IC16A.I0, IC4A.I0, IC8A.QA
- new net N$68: IC5A.I2, IC8B.QC
- new net N$69: IC5A.I1, IC8B.QB
- new net N$70: IC15A.I0, IC5A.I0, IC8B.QA
- new net N$71: IC14A.I1, IC3A.I3, IC9A.QD
- new net N$72: IC3A.I2, IC9A.QC
- new net N$73: IC3A.I1, IC9A.QB
- new net N$74: IC14A.I0, IC3A.I0, IC9A.QA
- new net N$75: IC13A.I1, IC2A.I3, IC9B.QD
- new net N$76: IC2A.I2, IC9B.QC
- new net N$77: IC13A.I0, IC2A.I1, IC9B.QB
- new net N$78: IC2A.I0, IC9B.QA
- new net N$79: IC10A.QD, IC12A.I1, IC7A.I3
- new net N$8: IC21A.Q, IC21B.CLK
- new net N$80: IC10A.QC, IC7A.I2
- new net N$81: IC10A.QB, IC11A.I0, IC12A.I0, IC7A.I1
- new net N$82: IC10A.QA, IC7A.I0
- new net N$83: IC10B.QD, IC6A.I3
- new net N$84: IC10B.QC, IC6A.I2
- new net N$85: IC10B.QB, IC6A.I1
- new net N$86: IC10B.QA, IC11A.I1, IC6A.I0
- new net N$87: D5.K, D7.A
- new net N$88: D8.K, D9.A
- new net N$89: IC17B.I1, IC21B.!Q, IC21B.D
- new net N$90: IC22A.!Q, IC22A.D
- new net N$91: IC17B.I3, IC22B.!Q, IC22B.D
- new net N$92: IC10B.A, IC12A.O
- new net N$93: IC18A.I0, IC23A.!Q, IC23A.D
- new net N$94: IC18A.I1, IC23B.!Q, IC23B.D
- new net N$95: IC18A.I3, IC24B.!Q, IC24B.D
- new net N$96: IC17A.I3, IC25A.!Q, IC25A.D
- new net N$97: IC25B.!Q, IC25B.D
- new net N$99: IC26B.!Q, IC26B.D
- net N$1: now also IC10A.A, IC13A.O; no longer C5.1, IC1.CON
- net N$10: now also IC21B.Q, IC22A.CLK; no longer C4.1, IC1.TRE, IC1.TRI, R4.2
- net N$11: now also IC17B.I2, IC22A.Q, IC22B.CLK; no longer D6.C, R1.2, T1.B
- net N$2: now also IC15A.I1, IC5A.I3, IC8B.QD; no longer FONTE_AC.2, TR1.2
- net N$3: now also IC15A.O, IC8A.A; no longer FONTE_AC.1, TR1.1
- net N$4: now also D5.A, R2.1; no longer D1.A, D3.C, TR1.4
- net N$5: now also D8.A, R1.1; no longer IC1./RES, IC1.VCC+, R3.2, T1.E
- net N$6: now also D12.A, IC19A.O; no longer IC1.DIS, R3.1, R4.1
- net N$7: now also IC20A.O, IC21A.CLK, S1.P; no longer D2.A, D4.C, TR1.3
- net N$9: now also CLOCLK_3600HZ.2, IC20A.I, S3.P; no longer C2.2, D1.C, D2.C, R1.1, T1.C
Other:
- moved on the sheet: R1

Commit message: chore
Parts:
- removed IC12, IC13, IC14, IC15, IC16: 74AHC1G08DCK, 74xx-little-us:74AHC1G08DCK
- IC1, IC11: value 74AHC1G08DCK -> 74AC08N; device 74xx-little-us:74AHC1G08DCK -> 74xx-eu:74AC08N
- IC10, IC8, IC9: value 74HC393D -> 74AC393N; device 74xx-eu:74HC393D -> 74xx-eu:74AC393N
- IC17, IC18: value 74AC21D -> 74AC21N; device 74xx-eu:74AC21D -> 74xx-eu:74AC21N
- IC20: value 4069D -> 4069N; device 40xx:4069D -> 40xx:4069N
- IC21, IC22, IC23, IC24, IC25, IC26: value 4013D -> 4013N; device 40xx:4013D -> 40xx:4013N
Connections:
- removed net N$107: R1.2, R2.2
- net N$1: now also IC1C.O; no longer IC13A.O
- net N$105: now also IC11B.I0, IC11B.I1; no longer IC1A.I0, IC1A.I1
- net N$111: now also IC11B.O; no longer IC11A.O
- net N$114: now also IC11A.O; no longer IC16A.O
- net N$117: now also IC1D.O; no longer IC14A.O
- net N$2: now also IC11C.I1; no longer IC15A.I1
- net N$3: now also IC11C.O; no longer IC15A.O
- net N$65: now also IC11A.I1; no longer IC16A.I1
- net N$66: now also IC11A.I0; no longer IC16A.I0
- net N$70: now also IC11C.I0; no longer IC15A.I0
- net N$71: now also IC1D.I1; no longer IC14A.I1
- net N$74: now also IC1D.I0; no longer IC14A.I0
- net N$75: now also IC1C.I1; no longer IC13A.I1
- net N$77: now also IC1C.I0; no longer IC13A.I0
- net N$79: now also IC1B.I1; no longer IC12A.I1
- net N$81: now also IC1A.I0, IC1B.I0; no longer IC11A.I0, IC12A.I0
- net N$86: now also IC1A.I1; no longer IC11A.I1
- net N$9: now also R1.2, R2.2
- net N$92: now also IC1B.O; no longer IC12A.O

Commit message: docs
Parts:
- removed DS1, DS2, DS3, DS4, DS5, DS6: ACSA56-51SUR, Display_LED:ACSA56-51SUR
- added LED1, LED2, LED3, LED4, LED5, LED6: S4301B, led-7-segment:S4301B
Connections:
- net N$113: now also LED1.C@1, LED1.C@2, LED2.C@1, LED2.C@2, LED3.C@1, LED3.C@2, LED4.C@1, LED4.C@2, LED5.C@1, LED5.C@2, LED6.C@1, LED6.C@2; no longer DS1.COM1, DS2.COM1, DS3.COM1, DS4.COM1, DS5.COM1, DS6.COM1
- net N$21: now also IC7A.G, LED6.G; no longer DS5.A, IC7A.A
- net N$22: now also IC7A.F, LED6.F; no longer DS5.B, IC7A.B
- net N$23: now also IC7A.E, LED6.E; no longer DS5.C, IC7A.C
- net N$24: now also LED6.D; no longer DS5.D
- net N$25: now also IC7A.C, LED6.C; no longer DS5.E, IC7A.E
- net N$26: now also IC7A.B, LED6.B; no longer DS5.G, IC7A.G
- net N$27: now also IC7A.A, LED6.A; no longer DS5.F, IC7A.F
- net N$28: now also LED1.A; no longer DS6.A
- net N$29: now also LED1.B; no longer DS6.B
- net N$30: now also LED1.C; no longer DS6.C
- net N$31: now also LED1.D; no longer DS6.D
- net N$32: now also LED1.E; no longer DS6.E
- net N$33: now also IC6A.F, LED1.F; no longer DS6.G, IC6A.G
- net N$34: now also IC6A.G, LED1.G; no longer DS6.F, IC6A.F
- net N$35: now also IC2A.G, LED5.G; no longer DS3.A, IC5A.A
- net N$36: now also IC2A.F, LED5.F; no longer DS3.B, IC5A.B
- net N$37: now also IC2A.E, LED5.E; no longer DS3.C, IC5A.C
- net N$38: now also IC2A.D, LED5.D; no longer DS3.D, IC5A.D
- net N$39: now also IC2A.C, LED5.C; no longer DS3.E, IC5A.E
- net N$40: now also IC2A.B, LED5.B; no longer DS3.G, IC5A.G
- net N$41: now also IC2A.A, LED5.A; no longer DS3.F, IC5A.F
- net N$42: now also IC3A.A, LED4.A; no longer DS4.A, IC4A.A
- net N$43: now also IC3A.B, LED4.B; no longer DS4.B, IC4A.B
- net N$44: now also IC3A.C, LED4.C; no longer DS4.C, IC4A.C
- net N$45: now also IC3A.D, LED4.D; no longer DS4.D, IC4A.D
- net N$46: now also IC3A.E, LED4.E; no longer DS4.E, IC4A.E
- net N$47: now also IC3A.F, LED4.F; no longer DS4.G, IC4A.G
- net N$48: now also IC3A.G, LED4.G; no longer DS4.F, IC4A.F
- net N$49: now also IC4A.G, LED3.G; no longer DS1.A, IC3A.A
- net N$50: now also IC4A.F, LED3.F; no longer DS1.B, IC3A.B
- net N$51: now also IC4A.E, LED3.E; no longer DS1.C, IC3A.C
- net N$52: now also IC4A.D, LED3.D; no longer DS1.D, IC3A.D
- net N$53: now also IC4A.C, LED3.C; no longer DS1.E, IC3A.E
- net N$54: now also IC4A.B, LED3.B; no longer DS1.G, IC3A.G
- net N$55: now also IC4A.A, LED3.A; no longer DS1.F, IC3A.F
- net N$56: now also IC5A.G, LED2.G; no longer DS2.A, IC2A.A
- net N$57: now also IC5A.F, LED2.F; no longer DS2.B, IC2A.B
- net N$58: now also IC5A.E, LED2.E; no longer DS2.C, IC2A.C
- net N$59: now also IC5A.D, LED2.D; no longer DS2.D, IC2A.D
- net N$60: now also IC5A.C, LED2.C; no longer DS2.E, IC2A.E
- net N$61: now also IC5A.B, LED2.B; no longer DS2.G, IC2A.G
- net N$62: now also IC5A.A, LED2.A; no longer DS2.F, IC2A.F
